File: ADCS board v1.6.kicad_pcb (KiCad board)
At the start: 2 copper layers, 95.9 x 90.2 mm, 18 parts, among them J1 Conn_02x30_Row_Letter_First, J2 Conn_02x30_Row_Letter_First, J3 Conn_01x05_Pin, J4 Conn_01x05_Pin, U1 4754

Commit message: redid the pcb based on schematic changes
Parts:
- added C1: C, Capacitor_SMD:C_0603_1608Metric, B.Cu at (76.5, 78.0)
- added C2: C, Capacitor_SMD:C_0603_1608Metric, B.Cu at (76.5, 80.5)
- moved J3 0.99 mm to (116.5, 107.4)
- moved G*** 0.21 mm to (100.5, 131.5)
Connections:
- net GPIO6 renamed IMU INT
- net GPIO8 renamed I2C0 SDA
- net GPIO9 renamed I2C0 SCL
- A1 pad 14: unconnected-(A1-GPIO10-Pad14) -> IMU RST
- A1 pad 19: GPIO14 -> OBC SDA
- A1 pad 20: GPIO15 -> OBC SCL
- A1 pad 21: GPIO16 -> GPS RXD
- A1 pad 22: GPIO17 -> GPS TXD
- J1 pad a1: unconnected-(J1-Pin_a1-Pada1) -> GND
- J1 pad a20: GPIO14 -> OBC SCL
- J1 pad a28: unconnected-(J1-Pin_a28-Pada28) -> GND
- J1 pad b20: GPIO15 -> OBC SDA
- J2 pad d27: unconnected-(J2-Pin_b27-Padd27) -> GND
- J3 pad 2: GPIO16 -> GPS TXD
- J3 pad 3: GPIO17 -> GPS RXD
- U1 pad JP2_2: unconnected-(U1-P0-PadJP2_2) -> GND
- U1 pad JP2_3: unconnected-(U1-P1-PadJP2_3) -> GND
- U1 pad JP2_4: unconnected-(U1-~{RST}-PadJP2_4) -> IMU RST
Routing:
- net OBC SDA: track 0.00 -> 52.8 mm
- net GPIO15: track 48.8 -> 0.00 mm
- net OBC SCL: track 0.00 -> 48.4 mm
- net GPIO14: track 45.6 -> 0.00 mm
- net IMU RST: track 0.00 -> 38.2 mm
- net GPIO17: track 27.0 -> 0.00 mm
- net GPIO16: track 13.3 -> 0.00 mm
- net GPS TXD: track 0.00 -> 11.4 mm
- net GPS RXD: track 0.00 -> 10.0 mm
- net /V_{IN}: track 137.2 -> 147.2 mm
- net +3.3V: track 177.7 -> 181.1 mm
- net GND: track 0.00 -> 1.93 mm, vias 3 -> 7
- net I2C0 SCL: track 76.1 -> 78.0 mm
- net I2C0 SDA: track 91.3 -> 93.2 mm
Other:
- board text added: "INT"
- board text added: "RST"
- board text added: "RX"
- board text added: "SCL"
- board text added: "SDA"
- board text added: "TX"
