File: ADCS board v1.6.kicad_sch (KiCad schematic)
At the start: 19 parts, among them J1 Conn_02x30_Row_Letter_First, J2 Conn_02x30_Row_Letter_First, J3 Conn_01x05_Pin, J4 Conn_01x05_Pin, U1 4754

Commit message: redid the pcb based on schematic changes
Connections:
- net GND: now also J1.a1 (Pin_a1), J1.a28 (Pin_a28), J2.d27 (Pin_b27), U1.JP2_2 (P0), U1.JP2_3 (P1)
- no-connect marks 31 -> 29
